File: IntelliMate/IntelliMate.kicad_sch (KiCad schematic)
At the start: 0 parts

Commit message: finished 0.1 design
Other:
- added sheet IR Beam (ir_beam.kicad_sch)
Changed lines of the file:
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@@
     (title "IntelliMate Prototype")
     (date "2023-05-23")
-    (rev "0")
+    (rev "0.1")
   )
   (wire (pts (xy 69.85 109.22) (xy 87.63 109.22))
@@
       )
     )
+  )
+  (sheet (at 160.02 74.93) (size 41.91 46.99) (fields_autoplaced)
+    (stroke (width 0.1524) (type solid))
+    (fill (color 0 0 0 0.0000))
+    (property "Sheetname" "IR Beam" (at 160.02 74.2184 0)
+      (effects (font (size 1.27 1.27)) (justify left bottom))
+    )
+    (property "Sheetfile" "ir_beam.kicad_sch" (at 160.02 122.5046 0)
+      (effects (font (size 1.27 1.27)) (justify left top))
+    )
+    (instances
+      (project "IntelliMate"
+        (path "/d2cbed07-112f-4ca6-afcf-4062e0b58893" (page "4"))
+      )
+    )
