File: IntelliMate/ir_beam.kicad_sch (KiCad schematic)
At the start: 16 parts, among them J11 Conn_01x03_Pin, Q18 BC547, Q19 BC547, Q20 BC547, U6 TSOP384xx

Commit message: added LEDs
Parts:
- C1: value C -> 0.1µ
- renumbered D120 to IR333-A1, D121 to IR333C1
Changed lines of the file:
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@@
       (effects (font (size 1.27 1.27)) (justify left))
     )
-    (property "Value" "C" (at 100.33 53.975 0)
+    (property "Value" "0.1µ" (at 100.33 53.975 0)
       (effects (font (size 1.27 1.27)) (justify left))
     )
@@
   (symbol (lib_id "Device:LED") (at 93.98 107.95 90) (unit 1)
     (in_bom yes) (on_board yes) (dnp no) (fields_autoplaced)
-    (property "Reference" "D121" (at 97.79 108.9025 90)
+    (property "Reference" "IR333C1" (at 97.79 108.9025 90)
       (effects (font (size 1.27 1.27)) (justify right))
     )
@@
       (project "IntelliMate"
         (path "/d2cbed07-112f-4ca6-afcf-4062e0b58893/a9279e42-41ff-46c0-91fb-0409ff955dc7"
-          (reference "D121") (unit 1)
+          (reference "IR333C1") (unit 1)
         )
       )
@@
   (symbol (lib_id "Device:LED") (at 93.98 97.79 90) (unit 1)
     (in_bom yes) (on_board yes) (dnp no) (fields_autoplaced)
-    (property "Reference" "D120" (at 97.79 98.7425 90)
+    (property "Reference" "IR333-A1" (at 97.79 98.7425 90)
       (effects (font (size 1.27 1.27)) (justify right))
     )
@@
       (project "IntelliMate"
         (path "/d2cbed07-112f-4ca6-afcf-4062e0b58893/a9279e42-41ff-46c0-91fb-0409ff955dc7"
-          (reference "D120") (unit 1)
-        )
-      )
+          (reference "IR333-A1") (unit 1)
+        )
+      )
