File: IntelliMate/power.kicad_sch (KiCad schematic)
At the start: 69 parts, among them J1 Conn_01x03_Socket, J8 Conn_01x08_Pin, J9 Conn_01x08_Pin, Q1 Q_NPN_Darlington_BCE, Q10 Q_NMOS_GDS, Q11 Q_NMOS_GDS, Q12 Q_NMOS_GDS, Q13 Q_NMOS_GDS, Q14 Q_NMOS_GDS, Q15 Q_NMOS_GDS, Q16 Q_NMOS_GDS, Q2 Q_PNP_Darlington_BCE, Q3 Q_PNP_Darlington_BCE, Q4 Q_PNP_Darlington_BCE, Q5 Q_PNP_Darlington_BCE, Q6 Q_PNP_Darlington_BCE, Q7 Q_PNP_Darlington_BCE, Q8 Q_NMOS_GDS, Q9 Q_NMOS_GDS, U1 LM723_DIP14, U2 ULN2803A, U3 LM301, U4 TBD62783A, U5 TBD62783A

Commit message: finished 0.1 design
Parts:
- C102, C103: value C -> 1µ
- C44: value C -> 0.1µ
- C9: value C -> 1p
Connections:
- net GND: now also J8.1 (Pin_1)
Changed lines of the file:
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@@
     (effects (font (size 1.27 1.27)) (justify left))
+  )
+  (symbol (lib_id "power:GND") (at 17.78 107.95 90) (unit 1)
+    (in_bom yes) (on_board yes) (dnp no) (fields_autoplaced)
+    (property "Reference" "#PWR029" (at 24.13 107.95 0)
+      (effects (font (size 1.27 1.27)) hide)
+    )
+    (property "Value" "GND" (at 21.59 108.585 90)
+      (effects (font (size 1.27 1.27)) (justify right))
+    )
+    (property "Footprint" "" (at 17.78 107.95 0)
+      (effects (font (size 1.27 1.27)) hide)
+    )
+    (property "Datasheet" "" (at 17.78 107.95 0)
+      (effects (font (size 1.27 1.27)) hide)
+    )
+    (pin "1")
+    (instances
+      (project "IntelliMate"
+        (path "/d2cbed07-112f-4ca6-afcf-4062e0b58893/5a0421ef-5bf1-40f6-9e02-e533a7a74d6f"
+          (reference "#PWR029") (unit 1)
+        )
+      )
+    )
   )
   (symbol (lib_id "Device:Q_NMOS_GDS") (at 135.89 162.56 270) (unit 1)
@@
       (effects (font (size 1.27 1.27)) (justify left))
     )
-    (property "Value" "C" (at 72.39 53.34 0)
+    (property "Value" "0.1µ" (at 69.85 53.34 0)
       (effects (font (size 1.27 1.27)) (justify left))
     )
@@
       (effects (font (size 1.27 1.27)) (justify left))
     )
-    (property "Value" "C" (at 115.57 64.135 0)
+    (property "Value" "1p" (at 115.57 64.135 0)
       (effects (font (size 1.27 1.27)) (justify left))
     )
@@
       (effects (font (size 1.27 1.27)) (justify right))
     )
-    (property "Value" "C" (at 254 64.135 0)
+    (property "Value" "1µ" (at 254 64.135 0)
       (effects (font (size 1.27 1.27)) (justify right))
     )
@@
       (effects (font (size 1.27 1.27)))
     )
-    (property "Value" "C" (at 254 29.21 90)
-      (effects (font (size 1.27 1.27)))
-    )
+    (property "Value" "1µ" (at 254 29.21 90)
+      (effects (font (size 1.27 1.27)))
+    )

Commit message: finished 0.1 design
Parts:
- C101, C110: value C_Polarized -> 6800µ
- C110: value C_Polarized -> 47µ
- C49: value C_Polarized -> 1000µ
Changed lines of the file:
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@@
       (effects (font (size 1.27 1.27)))
     )
-    (property "Value" "C_Polarized" (at 190.119 54.61 90)
+    (property "Value" "6800µ" (at 190.119 54.61 90)
       (effects (font (size 1.27 1.27)))
     )
@@
       (effects (font (size 1.27 1.27)) (justify left))
     )
-    (property "Value" "C_Polarized" (at 137.16 71.12 0)
+    (property "Value" "47µ" (at 137.16 71.12 0)
       (effects (font (size 1.27 1.27)) (justify left))
     )
@@
       (effects (font (size 1.27 1.27)))
     )
-    (property "Value" "C_Polarized" (at 190.119 26.67 90)
+    (property "Value" "1000µ" (at 190.119 26.67 90)
       (effects (font (size 1.27 1.27)))
     )
@@
       (effects (font (size 1.27 1.27)))
     )
-    (property "Value" "C_Polarized" (at 190.119 40.64 90)
-      (effects (font (size 1.27 1.27)))
-    )
+    (property "Value" "6800µ" (at 190.119 40.64 90)
+      (effects (font (size 1.27 1.27)))
+    )

Commit message: added LEDs
Parts:
- added D118, D119, D120, D121, D122, D123: LARGE LED, symbol Device:LED
- added D124, D125, D126, D127, D128, D129, D130, D131, D132: LED, symbol Device:LED
- added R33, R34, R35, R36, R37, R38: 10k, symbol Device:R
- added R39, R40, R47, R48, R49, R50, R51, R52, R53: 1k, symbol Device:R
- C43: value C -> 100p
Connections:
- net GND: now also D118.1 (K), D119.1 (K), D120.1 (K), D121.1 (K), D122.1 (K), D123.1 (K), D124.1 (K), D125.1 (K), D126.1 (K), D127.1 (K), D128.1 (K), D129.1 (K), D130.1 (K), D131.1 (K), D132.1 (K)
- net Q1: now also R38.2
- net Q10: now also R48.2
- net Q11: now also R49.2
- net Q12: now also R50.2
- net Q13: now also R51.2
- net Q14: now also R52.2
- net Q15: now also R53.2
- net Q2: now also R37.2
- net Q3: now also R36.2
- net Q4: now also R35.2
- net Q5: now also R34.2
- net Q6: now also R33.2
- net Q7: now also R39.2
- net Q8: now also R40.2
- net Q9: now also R47.2
- new net: D123.2 (A), R38.1
- new net: D118.2 (A), R33.1
- new net: D126.2 (A), R47.1
- new net: D121.2 (A), R36.1
- new net: D129.2 (A), R50.1
- new net: D131.2 (A), R52.1
- new net: D124.2 (A), R39.1
- new net: D120.2 (A), R35.1
- new net: D130.2 (A), R51.1
- new net: D127.2 (A), R48.1
- new net: D122.2 (A), R37.1
- new net: D119.2 (A), R34.1
- new net: D128.2 (A), R49.1
- new net: D132.2 (A), R53.1
- new net: D125.2 (A), R40.1
Other:
- moved on the sheet: Q13, Q15, R20, R21, R24, R25
