File: Dixie/Dixie.kicad_sch (KiCad schematic)
At the start: 0 parts

Commit message: setup new pcb design project
Other:
- title: IntelliMate Prototype -> Dixie VCU
Changed lines of the file:
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@@
   (paper "A4")
   (title_block
-    (title "IntelliMate Prototype")
+    (title "Dixie VCU")
     (date "2023-05-15")
     (rev "0")
@@
     )
     (instances
-      (project "IntelliMate"
+      (project "Dixie"
         (path "/d2cbed07-112f-4ca6-afcf-4062e0b58893" (page "2"))
       )
@@
     )
     (instances
-      (project "IntelliMate"
+      (project "Dixie"
         (path "/d2cbed07-112f-4ca6-afcf-4062e0b58893" (page "3"))
       )
