File: Dixie/actuators.kicad_sch (KiCad schematic)
At the start: 120 parts, among them J2 Conn_01x10_Pin, J3 Conn_01x10_Pin, J4 Conn_01x10_Pin, J5 Conn_01x10_Pin, J6 Conn_01x10_Pin, J7 Conn_01x10_Pin

Commit message: finished dixie pcb
Connections:
- net Q5: now reaches D80.1 (K), D82.2 (A), D84.2 (A), D86.2 (A), D88.2 (A), D90.2 (A), D92.2 (A), D94.2 (A), D96.2 (A), D98.2 (A), J6.10 (Pin_10)
- net Q7: now reaches D40.1 (K)
- net Q7: now also D100.1 (K), D12.1 (K), D59.1 (K), D78.1 (K), D81.1 (K)
- net Q15: now reaches D4.1 (K)
- net Q15: now also D116.1 (K), D24.1 (K), D43.1 (K), D62.1 (K), D97.1 (K)
- net Q2: now reaches D23.2 (A), D25.2 (A), D27.2 (A), D29.2 (A), D31.2 (A), D33.2 (A), D35.2 (A), D37.2 (A), D39.2 (A), D41.1 (K), J3.10 (Pin_10)
- net Q3: now reaches D61.2 (A), D63.2 (A), D65.2 (A), D67.2 (A), D69.2 (A), D71.2 (A), D73.2 (A), D75.2 (A), D77.2 (A), D79.1 (K), J5.10 (Pin_10)
- net Q4: now reaches D42.2 (A), D44.2 (A), D46.2 (A), D48.2 (A), D50.2 (A), D52.2 (A), D54.2 (A), D56.2 (A), D58.2 (A), D60.1 (K), J4.10 (Pin_10)
- net Q14: now reaches D114.1 (K)
- net Q14: now also D26.1 (K), D45.1 (K), D5.1 (K), D64.1 (K), D95.1 (K)
- net Q6: now reaches D101.2 (A), D103.2 (A), D105.2 (A), D107.2 (A), D109.2 (A), D111.2 (A), D113.2 (A), D115.2 (A), D117.2 (A), D99.1 (K), J7.10 (Pin_10)
- net Q1: now reaches D13.2 (A), D14.2 (A), D15.2 (A), D16.2 (A), D17.2 (A), D18.2 (A), D19.2 (A), D20.2 (A), D21.2 (A), D22.1 (K), J2.10 (Pin_10)
- net Q12: now reaches D7.1 (K)
- net Q12: now also D110.1 (K), D30.1 (K), D49.1 (K), D68.1 (K), D91.1 (K)
- net Q8: now reaches D57.1 (K)
- net Q8: now also D102.1 (K), D11.1 (K), D38.1 (K), D76.1 (K), D83.1 (K)
- net Q9: now reaches D74.1 (K)
- net Q9: now also D10.1 (K), D104.1 (K), D36.1 (K), D55.1 (K), D85.1 (K)
- net Q11: now reaches D8.1 (K)
- net Q11: now also D108.1 (K), D32.1 (K), D51.1 (K), D70.1 (K), D89.1 (K)
- net Q13: now reaches D66.1 (K)
- net Q13: now also D112.1 (K), D28.1 (K), D47.1 (K), D6.1 (K), D93.1 (K)
- net Q10: now reaches D34.1 (K)
- net Q10: now also D106.1 (K), D53.1 (K), D72.1 (K), D87.1 (K), D9.1 (K)
