File: Dixie/power.kicad_sch (KiCad schematic)
At the start: 61 parts, among them IC1 UDN2982LW, IC2 UDN2982LW, J1 Conn_01x03_Socket, Q1 Q_NPN_Darlington_BCE, Q10 Q_NMOS_GDS, Q11 Q_NMOS_GDS, Q12 Q_NMOS_GDS, Q13 Q_NMOS_GDS, Q14 Q_NMOS_GDS, Q15 Q_NMOS_GDS, Q16 Q_NMOS_GDS, Q2 Q_PNP_Darlington_BCE, Q3 Q_PNP_Darlington_BCE, Q4 Q_PNP_Darlington_BCE, Q5 Q_PNP_Darlington_BCE, Q6 Q_PNP_Darlington_BCE, Q7 Q_PNP_Darlington_BCE, Q8 Q_NMOS_GDS, Q9 Q_NMOS_GDS, U1 LM723_DIP14, U2 ULN2803A

Commit message: finished dixie pcb
Parts:
- added C110: C_Polarized, symbol Device:C_Polarized
- added C9: C, symbol Device:C
- added R29: 100, symbol Device:R
- added R30: 51.1, symbol Device:R
- added R31: 2.43k, symbol Device:R
- added R32: 7.52k, symbol Device:R
- added U3: LM301, symbol Amplifier_Operational:LM301
- R1: value R -> 1k
- R10, R11, R12, R13, R14, R15, R16, R17, R18, R19, R20, R21, R22, R23, R24, R25, R26, R27: value R -> 4.7k
- R2: value R -> 39.2k
- R3: value R -> 100
- R4, R5, R6, R7, R8, R9: value R -> 6.8k
- R51: value R -> 1.87k
Connections:
- net Earth is gone; now on net NEUT: D1.2 (A), J1.3 (Pin_3)
- net GND: now also Q10.3 (S), Q11.3 (S), Q12.3 (S), Q13.3 (S), Q14.3 (S), Q15.3 (S), Q16.3 (S), Q8.3 (S), Q9.3 (S), R10.2, R13.2, R15.2, R17.2, R19.2, R21.1, R23.2, R25.2, R27.2, U1.7 (V-), C110.2, R31.2, U3.4 (V-); no longer R2.2, R3.2, U1.2 (ILIM), U1.3 (CSEN)
- net LINE: now also C103.1, D101.2, D104.2, J1.2 (Pin_2)
- net NEUT: no longer C103.1, D101.2, D104.2, J1.2 (Pin_2)
- net Q10: now reaches Q11.2 (D)
- net Q10: no longer R17.2
- net at R1.2, R2.1: now also U3.2 (-)
- net at U2.10 (COM): now also IC1.9 (VS), IC2.9 (VS), Q2.3 (E), Q3.3 (E), Q4.3 (E), Q5.3 (E), Q6.3 (E), Q7.3 (E), XICON.1, C110.1, R29.1, R32.2, U3.3 (+)
- net Q11: now reaches Q12.2 (D)
- net Q11: no longer R19.2
- net at C43.1, U1.4 (-): now also R31.1, R32.1
- net Q15: now reaches Q16.2 (D)
- net Q15: no longer R27.2
- net at C49.1, D101.1 (+), Q1.2 (C)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: now also R29.2, R30.1
- net Q6: now reaches Q7.2 (C)
- net Q7: now reaches Q8.2 (D)
- net Q7: no longer R10.2
- net Q9: now reaches Q10.2 (D)
- net Q9: no longer R15.2
- net Q4: now reaches Q5.2 (C)
- net at Q13.1 (G), R20.2: now also R21.2; no longer R21.1
- net Q8: now reaches Q9.2 (D)
- net Q8: no longer R13.2
- net Q13: now reaches Q14.2 (D)
- net Q13: no longer R23.2
- net Q12: now reaches Q13.2 (D)
- net Q12: no longer R21.2
- net at Q1.3 (E), XICON.2: now also R1.1, R3.2, U1.2 (ILIM), U1.3 (CSEN), R30.2, U3.7 (V+)
- net Q5: now reaches Q6.2 (C)
- net Q3: now reaches Q4.2 (C)
- net Q14: now reaches Q15.2 (D)
- net Q14: no longer R25.2
- net at IC2.10 (NC_1): now also IC1.10 (NC_1)
- net Q2: now reaches Q3.2 (C)
- net Q1: now reaches Q2.2 (C)
- removed net LOGIC: R1.1, U1.7 (V-)
- new net: C9.1, U3.1 (BAL)
- new net: C9.2, U3.8 (C/B)
- new net: R2.2, U3.6
Other:
- moved on the sheet: C1, C101, C102, C103, C110, C43, C44, C49, D1, D101, D104, J1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

Commit message: setup new pcb design project
Parts:
- removed C1: C, symbol Device:C
